File: PCB/Pi_Pico_Zero_CMSIS_DAP.kicad_sch (KiCad schematic)
At the start: 8 parts, among them J1 CONN_PROG, J2 CONN_UART, U1 Pi_Pico_Zero

Commit message: MkI PCB Final
Other:
- title: (none) -> Pi Pico Zero CMSIS-DAP
Changed lines of the file:
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@@
 	(generator_version "8.0")
 	(paper "A4")
+	(title_block
+		(title "Pi Pico Zero CMSIS-DAP")
+		(date "2024-11-20")
+		(rev "MkI")
+		(comment 1 "ADBeta")
+	)
 	(junction
 		(at 267.97 19.685)
