File: PCB/Pico-DAP-Zero/Pico-DAP-Zero.kicad_sch (KiCad schematic)
At the start: 8 parts, among them J1 CONN_PROG, J2 CONN_UART, U1 Pi_Pico_Zero

Commit message: Renamed PCB
Other:
- company: (none) -> ADBeta
- title: Pi Pico Zero CMSIS-DAP -> Pico-DAP-Zero
- moved on the sheet: J1, J2, U1
