File: PCB/Pico-DAP-Zero/Pico-DAP-Zero.kicad_pcb (KiCad board)
At the start: 2 copper layers, 24 x 37.5 mm, 8 parts, among them J1 CONN_PROG, J2 CONN_UART, U1 Pi_Pico_Zero

Commit message: Changed PCB Silkscreen
Other:
- board text added: "Pico-DAP Zero MkI Nov 2024"
- board text removed: "Pi Pico Zero CMSIS-DAP MkI Nov 2024"
